Commit message: mecanum control

File: pdor_description/urdf/platform.macro.xacro (robot description, xacro)
@@ -88,5 +88,5 @@
 </link>
 <link name="${prefix}back_axis"/>
-<link name="${prefix}wheel_back_right">
+<link name="${prefix}wheel_rear_right">
   <visual>
     <geometry>
@@ -101,5 +101,5 @@
   </collision>
 </link>
-<link name="${prefix}wheel_back_left">
+<link name="${prefix}wheel_rear_left">
   <visual>
     <geometry>
@@ -114,10 +114,10 @@
   </collision>
 </link>
-<joint name="move_front_axis" type="fixed">
+<joint name="${prefix}move_front_axis" type="fixed">
   <parent link="${prefix}base_footprint"/>
   <child link="${prefix}front_axis"/>
   <origin xyz="${1.270/2 - 0.20} ${0.0} ${0.10}"/>
 </joint>
-<joint name="wheel_front_right_joint" type="continuous">
+<joint name="${prefix}wheel_front_right_joint" type="continuous">
   <parent link="${prefix}front_axis"/>
   <child link="${prefix}wheel_front_right"/>
@@ -125,5 +125,5 @@
   <origin xyz="0.0 ${-0.730/2 + 0.100/2 - 0.025} 0.0" rpy="${pi/2} 0.0 0.0"/>
 </joint>
-<joint name="wheel_front_left_joint" type="continuous">
+<joint name="${prefix}wheel_front_left_joint" type="continuous">
   <parent link="${prefix}front_axis"/>
   <child link="${prefix}wheel_front_left"/>
@@ -131,18 +131,18 @@
   <origin xyz="0.0 ${0.730/2 - 0.100/2 + 0.025} 0.0" rpy="${-pi/2} 0.0 0.0"/>
 </joint>
-<joint name="move_back_axis" type="fixed">
+<joint name="${prefix}move_rear_axis" type="fixed">
   <parent link="${prefix}base_footprint"/>
   <child link="${prefix}back_axis"/>
   <origin xyz="${-1.270/2 + 0.20} ${0.0} ${0.10}"/>
 </joint>
-<joint name="wheel_back_right_joint" type="continuous">
+<joint name="${prefix}wheel_rear_right_joint" type="continuous">
   <parent link="${prefix}back_axis"/>
-  <child link="${prefix}wheel_back_right"/>
+  <child link="${prefix}wheel_rear_right"/>
   <axis xyz="0 0 1"/>
   <origin xyz="0.0 ${-0.730/2 + 0.100/2 - 0.025} 0.0" rpy="${pi/2} 0.0 0.0"/>
 </joint>
-<joint name="wheel_back_left_joint" type="continuous">
+<joint name="${prefix}wheel_rear_left_joint" type="continuous">
   <parent link="${prefix}back_axis"/>
-  <child link="${prefix}wheel_back_left"/>
+  <child link="${prefix}wheel_rear_left"/>
   <axis xyz="0 0 1"/>
   <origin xyz="0.0 ${0.730/2 - 0.100/2 + 0.025} 0.0" rpy="${-pi/2} 0.0 0.0"/>

File: pdor_description/urdf/platform.ros2_control.xacro (robot description, xacro)
@@ -1,67 +1,69 @@
 <?xml version="1.0"?>
 <robot name = "platform" xmlns:xacro="http://www.ros.org/wiki/xacro">
-    <ros2_control name="platform" type="system">
-        <hardware>
-            <plugin>ethercat_driver/EthercatDriver</plugin>
-            <param name="master_id">0</param>
-            <param name="control_frequency">1000</param>
-        </hardware>
-        <joint name="joint_1">
-            <state_interface name="position"/>
-            <state_interface name="velocity"/>
-            <state_interface name="effort"/>
-            <command_interface name="velocity"/>
-            <command_interface name="reset_fault"/>
-            <ec_module name="ELMO">
-                <plugin>ethercat_generic_plugins/EcCiA402Drive</plugin>
-                <param name="alias">0</param>
-                <param name="position">0</param>
-                <param name="mode_of_operation">9</param>
-                <param name="slave_config">$(find pdor_description)/config/elmo_sx.yaml</param>
-            </ec_module>
-        </joint>
-        <joint name="joint_2">
-            <state_interface name="position"/>
-            <state_interface name="velocity"/>
-            <state_interface name="effort"/>
-            <command_interface name="velocity"/>
-            <command_interface name="reset_fault"/>
-            <ec_module name="ELMO">
-                <plugin>ethercat_generic_plugins/EcCiA402Drive</plugin>
-                <param name="alias">0</param>
-                <param name="position">1</param>
-                <param name="mode_of_operation">9</param>
-                <param name="slave_config">$(find pdor_description)/config/elmo_dx.yaml</param>
-            </ec_module>
-        </joint>
-        <joint name="joint_3">
-            <state_interface name="position"/>
-            <state_interface name="velocity"/>
-            <state_interface name="effort"/>
-            <command_interface name="velocity"/>
-            <command_interface name="reset_fault"/>
-            <ec_module name="ELMO">
-                <plugin>ethercat_generic_plugins/EcCiA402Drive</plugin>
-                <param name="alias">0</param>
-                <param name="position">2</param>
-                <param name="mode_of_operation">9</param>
-                <param name="slave_config">$(find pdor_description)/config/elmo_dx.yaml</param>
-            </ec_module>
-        </joint>
-        <joint name="joint_4">
-            <state_interface name="position"/>
-            <state_interface name="velocity"/>
-            <state_interface name="effort"/>
-            <command_interface name="velocity"/>
-            <command_interface name="reset_fault"/>
-            <ec_module name="ELMO">
-                <plugin>ethercat_generic_plugins/EcCiA402Drive</plugin>
-                <param name="alias">0</param>
-                <param name="position">3</param>
-                <param name="mode_of_operation">9</param>
-                <param name="slave_config">$(find pdor_description)/config/elmo_encoder_2000.yaml</param>
-            </ec_module>
-        </joint>
-    </ros2_control>
+    <xacro:macro name="platform_ros2_control" params="prefix">
+        <ros2_control name="platform" type="system">
+            <hardware>
+                <plugin>ethercat_driver/EthercatDriver</plugin>
+                <param name="master_id">0</param>
+                <param name="control_frequency">1000</param>
+            </hardware>
+            <joint name="${prefix}wheel_front_left_joint">
+                <state_interface name="position"/>
+                <state_interface name="velocity"/>
+                <state_interface name="effort"/>
+                <command_interface name="velocity"/>
+                <command_interface name="reset_fault"/>
+                <ec_module name="ELMO">
+                    <plugin>ethercat_generic_plugins/EcCiA402Drive</plugin>
+                    <param name="alias">0</param>
+                    <param name="position">0</param>
+                    <param name="mode_of_operation">9</param>
+                    <param name="slave_config">$(find pdor_description)/config/elmo_sx.yaml</param>
+                </ec_module>
+            </joint>
+            <joint name="${prefix}wheel_front_right_joint">
+                <state_interface name="position"/>
+                <state_interface name="velocity"/>
+                <state_interface name="effort"/>
+                <command_interface name="velocity"/>
+                <command_interface name="reset_fault"/>
+                <ec_module name="ELMO">
+                    <plugin>ethercat_generic_plugins/EcCiA402Drive</plugin>
+                    <param name="alias">0</param>
+                    <param name="position">1</param>
+                    <param name="mode_of_operation">9</param>
+                    <param name="slave_config">$(find pdor_description)/config/elmo_dx.yaml</param>
+                </ec_module>
+            </joint>
+            <joint name="${prefix}wheel_rear_right_joint">
+                <state_interface name="position"/>
+                <state_interface name="velocity"/>
+                <state_interface name="effort"/>
+                <command_interface name="velocity"/>
+                <command_interface name="reset_fault"/>
+                <ec_module name="ELMO">
+                    <plugin>ethercat_generic_plugins/EcCiA402Drive</plugin>
+                    <param name="alias">0</param>
+                    <param name="position">2</param>
+                    <param name="mode_of_operation">9</param>
+                    <param name="slave_config">$(find pdor_description)/config/elmo_dx.yaml</param>
+                </ec_module>
+            </joint>
+            <joint name="${prefix}wheel_rear_left_joint">
+                <state_interface name="position"/>
+                <state_interface name="velocity"/>
+                <state_interface name="effort"/>
+                <command_interface name="velocity"/>
+                <command_interface name="reset_fault"/>
+                <ec_module name="ELMO">
+                    <plugin>ethercat_generic_plugins/EcCiA402Drive</plugin>
+                    <param name="alias">0</param>
+                    <param name="position">3</param>
+                    <param name="mode_of_operation">9</param>
+                    <param name="slave_config">$(find pdor_description)/config/elmo_encoder_2000.yaml</param>
+                </ec_module>
+            </joint>
+        </ros2_control>
+    </xacro:macro>
 </robot>
 <!--

File: pdor_description/urdf/platform.urdf.xacro (robot description, xacro)
@@ -2,8 +2,8 @@
 <!-- Scara manipulator -->
 <robot xmlns:xacro="http://www.ros.org/wiki/xacro" name="pdor_platform">
-    <!-- Import scara urdf file -->
-    <xacro:include filename="$(find pdor_description)/urdf/platform.urdf" />
-    <xacro:pdor_base prefix=""/>
-    <!-- Import scara ros2_control description -->
-    <!-- <xacro:include filename="$(find pdor_description)/urdf/platform.ros2_control.xacro" /> -->
+    <xacro:arg name="prefix" default=""/>
+    <xacro:include filename="$(find pdor_description)/urdf/platform.macro.xacro" />
+    <xacro:pdor_base prefix="$(arg prefix)"/>
+    <xacro:include filename="$(find pdor_description)/urdf/platform.ros2_control.xacro" />
+    <xacro:platform_ros2_control prefix="$(arg prefix)"/>
 </robot>

Commit message: fix

File: pdor_description/urdf/platform.macro.xacro (robot description, xacro)
@@ -123,5 +123,5 @@
   <child link="${prefix}wheel_front_right"/>
   <axis xyz="0 0 1"/>
-  <origin xyz="0.0 ${-0.730/2 + 0.100/2 - 0.025} 0.0" rpy="${pi/2} 0.0 0.0"/>
+  <origin xyz="0.0 ${-0.730/2 + 0.100/2} 0.0" rpy="${pi/2} 0.0 0.0"/>
 </joint>
 <joint name="${prefix}wheel_front_left_joint" type="continuous">
@@ -129,5 +129,5 @@
   <child link="${prefix}wheel_front_left"/>
   <axis xyz="0 0 1"/>
-  <origin xyz="0.0 ${0.730/2 - 0.100/2 + 0.025} 0.0" rpy="${-pi/2} 0.0 0.0"/>
+  <origin xyz="0.0 ${0.730/2 - 0.100/2} 0.0" rpy="${-pi/2} 0.0 0.0"/>
 </joint>
 <joint name="${prefix}move_rear_axis" type="fixed">
@@ -140,5 +140,5 @@
   <child link="${prefix}wheel_rear_right"/>
   <axis xyz="0 0 1"/>
-  <origin xyz="0.0 ${-0.730/2 + 0.100/2 - 0.025} 0.0" rpy="${pi/2} 0.0 0.0"/>
+  <origin xyz="0.0 ${-0.730/2 + 0.100/2} 0.0" rpy="${pi/2} 0.0 0.0"/>
 </joint>
 <joint name="${prefix}wheel_rear_left_joint" type="continuous">
@@ -146,5 +146,5 @@
   <child link="${prefix}wheel_rear_left"/>
   <axis xyz="0 0 1"/>
-  <origin xyz="0.0 ${0.730/2 - 0.100/2 + 0.025} 0.0" rpy="${-pi/2} 0.0 0.0"/>
+  <origin xyz="0.0 ${0.730/2 - 0.100/2} 0.0" rpy="${-pi/2} 0.0 0.0"/>
 </joint>
 </xacro:macro>

Commit message: fix

File: pdor_description/urdf/platform.macro.xacro (robot description, xacro)
@@ -148,4 +148,11 @@
   <origin xyz="0.0 ${0.730/2 - 0.100/2} 0.0" rpy="${-pi/2} 0.0 0.0"/>
 </joint>
+<!-- Lidar -->
+<link name="${prefix}lidar"/>
+<joint name="core_to_lidar" type="fixed">
+  <parent link="${prefix}front_axis"/>
+  <child link="${prefix}lidar"/>
+  <origin xyz="0 0 ${0.35}"/>
+</joint>
 </xacro:macro>
 </robot>

Commit message: fix

File: pdor_description/urdf/platform.macro.xacro (robot description, xacro)
@@ -153,5 +153,5 @@
   <parent link="${prefix}front_axis"/>
   <child link="${prefix}lidar"/>
-  <origin xyz="0 0 ${0.35}"/>
+  <origin xyz="0 0 ${0.35}" rpy="0.0 0.0 ${-pi/2}"/>
 </joint>
 </xacro:macro>

Commit message: urdf fix

File: pdor_description/urdf/platform.macro.xacro (robot description, xacro)
@@ -122,5 +122,5 @@
   <parent link="${prefix}front_axis"/>
   <child link="${prefix}wheel_front_right"/>
-  <axis xyz="0 0 1"/>
+  <axis xyz="0 0 -1"/>
   <origin xyz="0.0 ${-0.730/2 + 0.100/2} 0.0" rpy="${pi/2} 0.0 0.0"/>
 </joint>
@@ -139,5 +139,5 @@
   <parent link="${prefix}back_axis"/>
   <child link="${prefix}wheel_rear_right"/>
-  <axis xyz="0 0 1"/>
+  <axis xyz="0 0 -1"/>
   <origin xyz="0.0 ${-0.730/2 + 0.100/2} 0.0" rpy="${pi/2} 0.0 0.0"/>
 </joint>

Commit message: add imm

File: pdor_description/urdf/platform.macro.xacro (robot description, xacro)
@@ -3,4 +3,10 @@
 <xacro:macro name="pdor_base" params="prefix">
   <link name="${prefix}base_footprint"/>
+  <link name="${prefix}mount_frame"/>
+  <joint name="mount_frame_joint" type="fixed">
+    <parent link="${prefix}base_footprint"/>
+    <child link="${prefix}mount_frame"/>
+    <origin xyz="0 0 ${0.290+0.310}"/>
+  </joint>
   <xacro:include filename="$(find pdor_description)/config/materials.urdf" />
 <!-- Base structure -->
