Commit message: rename

File: grond_description/urdf/platform.macro.xacro (robot description, xacro)
@@ -1,5 +1,5 @@
 <?xml version = "1.0"?>
 <robot name = "platform" xmlns:xacro="http://www.ros.org/wiki/xacro">
-<xacro:macro name="pdor_base" params="prefix">
+<xacro:macro name="grond_base" params="prefix">
   <link name="${prefix}base_footprint"/>
   <link name="${prefix}mount_frame"/>
@@ -9,5 +9,5 @@
     <origin xyz="0 0 ${0.290+0.310}"/>
   </joint>
-  <xacro:include filename="$(find pdor_description)/config/materials.urdf" />
+  <xacro:include filename="$(find grond_description)/config/materials.urdf" />
 <!-- Base structure -->
   <link name="${prefix}core">

File: grond_description/urdf/platform.ros2_control.xacro (robot description, xacro)
@@ -19,5 +19,5 @@
                     <param name="position">0</param>
                     <param name="mode_of_operation">9</param>
-                    <param name="slave_config">$(find pdor_description)/config/elmo_sx.yaml</param>
+                    <param name="slave_config">$(find grond_description)/config/elmo_sx.yaml</param>
                 </ec_module>
             </joint>
@@ -33,5 +33,5 @@
                     <param name="position">1</param>
                     <param name="mode_of_operation">9</param>
-                    <param name="slave_config">$(find pdor_description)/config/elmo_dx.yaml</param>
+                    <param name="slave_config">$(find grond_description)/config/elmo_dx.yaml</param>
                 </ec_module>
             </joint>
@@ -47,5 +47,5 @@
                     <param name="position">2</param>
                     <param name="mode_of_operation">9</param>
-                    <param name="slave_config">$(find pdor_description)/config/elmo_dx.yaml</param>
+                    <param name="slave_config">$(find grond_description)/config/elmo_dx.yaml</param>
                 </ec_module>
             </joint>
@@ -61,5 +61,5 @@
                     <param name="position">3</param>
                     <param name="mode_of_operation">9</param>
-                    <param name="slave_config">$(find pdor_description)/config/elmo_encoder_2000.yaml</param>
+                    <param name="slave_config">$(find grond_description)/config/elmo_encoder_2000.yaml</param>
                 </ec_module>
             </joint>

File: grond_description/urdf/system.urdf.xacro (robot description, xacro)
@@ -1,5 +1,5 @@
 <?xml version = "1.0"?>
 <robot name = "lampo_imm" xmlns:xacro="http://www.ros.org/wiki/xacro">
-  <xacro:include filename="$(find pdor_description)/urdf/system.xacro"/>
+  <xacro:include filename="$(find grond_description)/urdf/system.xacro"/>
   <xacro:lampo_imm prefix="lampo/" generate_ros2_control_tag="true"/>
 </robot>

File: grond_description/urdf/system.xacro (robot description, xacro)
@@ -3,8 +3,8 @@
   <xacro:macro name="lampo_imm" params="prefix generate_ros2_control_tag">
     <xacro:include filename="$(find ur_description)/urdf/ur_macro.xacro"/>
-    <xacro:include filename="$(find pdor_description)/urdf/platform.macro.xacro"/>
-    <xacro:pdor_base prefix="${prefix}"/>
+    <xacro:include filename="$(find grond_description)/urdf/platform.macro.xacro"/>
+    <xacro:grond_base prefix="${prefix}"/>
     <xacro:if value="${generate_ros2_control_tag}">
-      <xacro:include filename="$(find pdor_description)/urdf/platform.ros2_control.xacro"/>
+      <xacro:include filename="$(find grond_description)/urdf/platform.ros2_control.xacro"/>
       <xacro:platform_ros2_control prefix="${prefix}"/>
     </xacro:if>
