Commit message: launch scan

File: grond_description/urdf/system.xacro (robot description, xacro)
@@ -1,5 +1,5 @@
 <?xml version = "1.0"?>
 <robot name = "lampo_imm_macro" xmlns:xacro="http://www.ros.org/wiki/xacro">
-  <xacro:macro name="lampo_imm" params="prefix generate_ros2_control_tag sim_gz:=false">
+  <xacro:macro name="lampo_imm" params="prefix generate_ros2_control_tag sim_gz:=false use_fake_ur:=false">
     <xacro:include filename="$(find ur_description)/urdf/ur_macro.xacro"/>
     <xacro:include filename="$(find grond_description)/urdf/platform.macro.xacro"/>
@@ -22,5 +22,5 @@
       safety_pos_margin="0.15"
       safety_k_position="20"
-      use_fake_hardware="false"
+      use_fake_hardware="${use_fake_ur}"
       fake_sensor_commands="false"
       sim_gazebo="$(arg sim_gz)"
@@ -37,8 +37,8 @@
       tool_device_name="/tmp/ttyUR"
       tool_tcp_port="54321"
-      robot_ip="0.0.0.0"
-      script_filename=""
-      output_recipe_filename=""
-      input_recipe_filename=""
+      robot_ip="192.168.10.2"
+      script_filename="/opt/ros/humble/share/ur_client_library/resources/external_control.urscript"
+      output_recipe_filename="/opt/ros/humble/share/ur_robot_driver/resources/rtde_output_recipe.txt"
+      input_recipe_filename="/opt/ros/humble/share/ur_robot_driver/resources/rtde_input_recipe.txt"
       reverse_port="50001"
       script_sender_port="50002"
