Commit message: add fake_base + fix admittance

File: grond_description/urdf/platform.ros2_control.xacro (robot description, xacro)
@@ -1,6 +1,7 @@
 <?xml version="1.0"?>
 <robot name = "platform" xmlns:xacro="http://www.ros.org/wiki/xacro">
-    <xacro:macro name="platform_ros2_control" params="prefix">
+    <xacro:macro name="platform_ros2_control" params="prefix use_fake_hardware">
         <ros2_control name="platform" type="system">
+          <xacro:unless value="${use_fake_hardware}">
             <hardware>
                 <plugin>ethercat_driver/EthercatDriver</plugin>
@@ -8,4 +9,10 @@
                 <param name="control_frequency">1000</param>
             </hardware>
+          </xacro:unless>
+          <xacro:if value="${use_fake_hardware}">
+            <hardware>
+              <plugin>mock_components/GenericSystem</plugin>
+            </hardware>
+          </xacro:if>
             <joint name="${prefix}wheel_front_left_joint">
                 <state_interface name="position"/>
@@ -13,12 +20,14 @@
                 <state_interface name="effort"/>
                 <command_interface name="velocity"/>
-                <command_interface name="reset_fault"/>
-                <ec_module name="ELMO">
-                    <plugin>ethercat_generic_plugins/EcCiA402Drive</plugin>
-                    <param name="alias">0</param>
-                    <param name="position">0</param>
-                    <param name="mode_of_operation">9</param>
-                    <param name="slave_config">$(find grond_description)/config/elmo_sx.yaml</param>
-                </ec_module>
+                <xacro:unless value="${use_fake_hardware}">
+                  <command_interface name="reset_fault"/>
+                  <ec_module name="ELMO">
+                      <plugin>ethercat_generic_plugins/EcCiA402Drive</plugin>
+                      <param name="alias">0</param>
+                      <param name="position">0</param>
+                      <param name="mode_of_operation">9</param>
+                      <param name="slave_config">$(find grond_description)/config/elmo_sx.yaml</param>
+                  </ec_module>
+                </xacro:unless>
             </joint>
             <joint name="${prefix}wheel_front_right_joint">
@@ -27,12 +36,14 @@
                 <state_interface name="effort"/>
                 <command_interface name="velocity"/>
-                <command_interface name="reset_fault"/>
-                <ec_module name="ELMO">
-                    <plugin>ethercat_generic_plugins/EcCiA402Drive</plugin>
-                    <param name="alias">0</param>
-                    <param name="position">1</param>
-                    <param name="mode_of_operation">9</param>
-                    <param name="slave_config">$(find grond_description)/config/elmo_dx.yaml</param>
-                </ec_module>
+                <xacro:unless value="${use_fake_hardware}">
+                  <command_interface name="reset_fault"/>
+                  <ec_module name="ELMO">
+                      <plugin>ethercat_generic_plugins/EcCiA402Drive</plugin>
+                      <param name="alias">0</param>
+                      <param name="position">1</param>
+                      <param name="mode_of_operation">9</param>
+                      <param name="slave_config">$(find grond_description)/config/elmo_dx.yaml</param>
+                  </ec_module>
+                </xacro:unless>
             </joint>
             <joint name="${prefix}wheel_rear_right_joint">
@@ -41,12 +52,14 @@
                 <state_interface name="effort"/>
                 <command_interface name="velocity"/>
-                <command_interface name="reset_fault"/>
-                <ec_module name="ELMO">
-                    <plugin>ethercat_generic_plugins/EcCiA402Drive</plugin>
-                    <param name="alias">0</param>
-                    <param name="position">2</param>
-                    <param name="mode_of_operation">9</param>
-                    <param name="slave_config">$(find grond_description)/config/elmo_dx.yaml</param>
-                </ec_module>
+                <xacro:unless value="${use_fake_hardware}">
+                  <command_interface name="reset_fault"/>
+                  <ec_module name="ELMO">
+                      <plugin>ethercat_generic_plugins/EcCiA402Drive</plugin>
+                      <param name="alias">0</param>
+                      <param name="position">2</param>
+                      <param name="mode_of_operation">9</param>
+                      <param name="slave_config">$(find grond_description)/config/elmo_dx.yaml</param>
+                  </ec_module>
+                </xacro:unless>
             </joint>
             <joint name="${prefix}wheel_rear_left_joint">
@@ -55,12 +68,14 @@
                 <state_interface name="effort"/>
                 <command_interface name="velocity"/>
-                <command_interface name="reset_fault"/>
-                <ec_module name="ELMO">
-                    <plugin>ethercat_generic_plugins/EcCiA402Drive</plugin>
-                    <param name="alias">0</param>
-                    <param name="position">3</param>
-                    <param name="mode_of_operation">9</param>
-                    <param name="slave_config">$(find grond_description)/config/elmo_encoder_2000.yaml</param>
-                </ec_module>
+                <xacro:unless value="${use_fake_hardware}">
+                  <command_interface name="reset_fault"/>
+                  <ec_module name="ELMO">
+                      <plugin>ethercat_generic_plugins/EcCiA402Drive</plugin>
+                      <param name="alias">0</param>
+                      <param name="position">3</param>
+                      <param name="mode_of_operation">9</param>
+                      <param name="slave_config">$(find grond_description)/config/elmo_encoder_2000.yaml</param>
+                  </ec_module>
+                </xacro:unless>
             </joint>
         </ros2_control>

File: grond_description/urdf/platform.urdf.xacro (robot description, xacro)
@@ -3,7 +3,8 @@
 <robot xmlns:xacro="http://www.ros.org/wiki/xacro" name="grond_platform">
     <xacro:arg name="prefix" default=""/>
+    <xacro:arg name="use_fake_hardware" default="false"/>
     <xacro:include filename="$(find grond_description)/urdf/platform.macro.xacro" />
     <xacro:grond_base prefix="$(arg prefix)"/>
     <xacro:include filename="$(find grond_description)/urdf/platform.ros2_control.xacro" />
-    <xacro:platform_ros2_control prefix="$(arg prefix)"/>
+    <xacro:platform_ros2_control prefix="$(arg prefix)" use_fake_hardware="$(arg use_fake_hardware)"/>
 </robot>

File: grond_description/urdf/system.urdf.xacro (robot description, xacro)
@@ -5,5 +5,6 @@
   <xacro:arg name="sim_gz" default="false"/>
   <xacro:arg name="use_fake_ur" default="false"/>
+  <xacro:arg name="use_fake_base" default="false"/>
   <xacro:include filename="$(find grond_description)/urdf/system.xacro"/>
-  <xacro:lampo_imm prefix="$(arg name)/" generate_ros2_control_tag="true" sim_gz="$(arg sim_gz)" use_fake_ur="$(arg use_fake_ur)"/>
+  <xacro:lampo_imm prefix="$(arg name)/" generate_ros2_control_tag="true" sim_gz="$(arg sim_gz)" use_fake_ur="$(arg use_fake_ur)" use_fake_base="$(arg use_fake_base)"/>
 </robot>

File: grond_description/urdf/system.xacro (robot description, xacro)
@@ -1,5 +1,5 @@
 <?xml version = "1.0"?>
 <robot name = "lampo_imm_macro" xmlns:xacro="http://www.ros.org/wiki/xacro">
-  <xacro:macro name="lampo_imm" params="prefix generate_ros2_control_tag sim_gz:=false use_fake_ur:=false">
+  <xacro:macro name="lampo_imm" params="prefix generate_ros2_control_tag sim_gz:=false use_fake_ur:=false use_fake_base:=false">
     <xacro:include filename="$(find ur_description)/urdf/ur_macro.xacro"/>
     <xacro:include filename="$(find grond_description)/urdf/platform.macro.xacro"/>
@@ -7,5 +7,5 @@
     <xacro:if value="${generate_ros2_control_tag}">
       <xacro:include filename="$(find grond_description)/urdf/platform.ros2_control.xacro"/>
-      <xacro:platform_ros2_control prefix="${prefix}"/>
+      <xacro:platform_ros2_control prefix="${prefix}" use_fake_hardware="${use_fake_base}"/>
     </xacro:if>
     <xacro:ur_robot
