Commit message: flag gz

File: grond_description/urdf/system.urdf.xacro (robot description, xacro)
@@ -3,5 +3,6 @@
   <xacro:arg name="name" default="lampo"/>
   <xacro:arg name="generate_ros2_control_tag" default="true"/>
+  <xacro:arg name="sim_gz" default="false"/>
   <xacro:include filename="$(find grond_description)/urdf/system.xacro"/>
-  <xacro:lampo_imm prefix="$(arg name)/" generate_ros2_control_tag="true"/>
+  <xacro:lampo_imm prefix="$(arg name)/" generate_ros2_control_tag="true" sim_gz="$(arg sim_gz)"/>
 </robot>

File: grond_description/urdf/system.xacro (robot description, xacro)
@@ -1,5 +1,5 @@
 <?xml version = "1.0"?>
 <robot name = "lampo_imm_macro" xmlns:xacro="http://www.ros.org/wiki/xacro">
-  <xacro:macro name="lampo_imm" params="prefix generate_ros2_control_tag">
+  <xacro:macro name="lampo_imm" params="prefix generate_ros2_control_tag sim_gz:=false">
     <xacro:include filename="$(find ur_description)/urdf/ur_macro.xacro"/>
     <xacro:include filename="$(find grond_description)/urdf/platform.macro.xacro"/>
@@ -24,5 +24,5 @@
       use_fake_hardware="false"
       fake_sensor_commands="false"
-      sim_gazebo="false"
+      sim_gazebo="$(arg sim_gz)"
       sim_ignition="false"
       headless_mode="false"

Commit message: various fix

File: grond_description/urdf/system.urdf.xacro (robot description, xacro)
@@ -7,4 +7,4 @@
   <xacro:arg name="use_fake_base" default="false"/>
   <xacro:include filename="$(find grond_description)/urdf/system.xacro"/>
-  <xacro:lampo_imm prefix="$(arg name)/" generate_ros2_control_tag="true" sim_gz="$(arg sim_gz)" use_fake_ur="$(arg use_fake_ur)" use_fake_base="$(arg use_fake_base)"/>
+  <xacro:lampo_imm prefix="$(arg name)/" generate_ros2_control_tag="$(arg generate_ros2_control_tag)" sim_gz="$(arg sim_gz)" use_fake_ur="$(arg use_fake_ur)" use_fake_base="$(arg use_fake_base)"/>
 </robot>

File: grond_description/urdf/system.xacro (robot description, xacro)
@@ -49,5 +49,5 @@
       keep_alive_count="2"
     >
-      <origin xyz="0 0 0" />
+      <origin xyz="0 0 0" rpy="0 0 ${-pi/2}" />
     </xacro:ur_robot>
   </xacro:macro>

Commit message: add headless ur

File: grond_description/urdf/system.urdf.xacro (robot description, xacro)
@@ -6,5 +6,6 @@
   <xacro:arg name="use_fake_ur" default="false"/>
   <xacro:arg name="use_fake_base" default="false"/>
+  <xacro:arg name="headless_ur" default="false"/>
   <xacro:include filename="$(find grond_description)/urdf/system.xacro"/>
-  <xacro:lampo_imm prefix="$(arg name)/" generate_ros2_control_tag="$(arg generate_ros2_control_tag)" sim_gz="$(arg sim_gz)" use_fake_ur="$(arg use_fake_ur)" use_fake_base="$(arg use_fake_base)"/>
+  <xacro:lampo_imm prefix="$(arg name)/" generate_ros2_control_tag="$(arg generate_ros2_control_tag)" sim_gz="$(arg sim_gz)" use_fake_ur="$(arg use_fake_ur)" use_fake_base="$(arg use_fake_base)" headless_ur="$(arg headless_ur)"/>
 </robot>

File: grond_description/urdf/system.xacro (robot description, xacro)
@@ -1,5 +1,5 @@
 <?xml version = "1.0"?>
 <robot name = "lampo_imm_macro" xmlns:xacro="http://www.ros.org/wiki/xacro">
-  <xacro:macro name="lampo_imm" params="prefix generate_ros2_control_tag sim_gz:=false use_fake_ur:=false use_fake_base:=false">
+  <xacro:macro name="lampo_imm" params="prefix generate_ros2_control_tag headless_ur:=false sim_gz:=false use_fake_ur:=false use_fake_base:=false">
     <xacro:include filename="$(find ur_description)/urdf/ur_macro.xacro"/>
     <xacro:include filename="$(find grond_description)/urdf/platform.macro.xacro"/>
@@ -26,5 +26,5 @@
       sim_gazebo="$(arg sim_gz)"
       sim_ignition="false"
-      headless_mode="false"
+      headless_mode="${headless_ur}"
       initial_positions="${dict(shoulder_pan_joint=0.0,shoulder_lift_joint=-1.57,elbow_joint=0.0,wrist_1_joint=-1.57,wrist_2_joint=0.0,wrist_3_joint=0.0)}"
       use_tool_communication="false"
